File: schematic & pcb/kicad_project/_carrier/_carrier.kicad_pcb (KiCad board)
At the start: 2 copper layers, 59.5 x 52.5 mm, 12 parts, among them J1 ANAL, J2 OCTSTP, J3 KB, J4 i2c, J5 UART, J6 xtr_GPIO, J7 xtr_VCC, J8 xtr_GND, U1 ProMicro

Commit message: keyboard pcb
Routing:
- net +5V: track 145.6 -> 146.2 mm
Other:
- board text added: "10"
- board text added: "16"
- board text added: "2"
- board text added: "3"
- board text added: "5"
- board text added: "6"
- board text added: "7"
- board text added: "A0"
- board text added: "A1"
- board text added: "A2"
- board text added: "A3"
- board text added: "Designed by Recsnik B. & Cserhegyi R."
- board text added: "ZAP"
- board text added: "killroy was here"
- board text removed: "+"
