File: schematic & pcb/kicad_project/custom_exports/mcu-kb-octstp-anal-combinedpcb/mkoa_combinedpcb.kicad_pcb (KiCad board)
At the start: 2 copper layers, 130.2 x 90.8 mm, 34 parts, among them J1 ANAL, J1 Conn_01x03_Socket, J1 Conn_01x05_Socket, J1 Conn_01x06_Socket, J2 Conn_01x08_Socket, J2 OCTSTP, J3 Conn_01x08_Socket, J3 KB, J4 Conn_01x08_Socket, J4 i2c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

Commit message: missed pushes
Other:
- board size 130.2 x 90.8 mm -> 130.2 x 93.2 mm
- board text removed: "+"
